Commit message: Diff_bot urdf visualization

File: description/base.xacro (robot description, xacro)
@@ -2,6 +2,6 @@
 <robot xmlns:xacro="http://www.ros.org/wiki/xacro">
   <!-- Variables -->
-  <xacro:property name="base_length" value="0.372"/>
-  <xacro:property name="base_width" value="0.361"/>
+  <xacro:property name="base_length" value="0.498"/>
+  <xacro:property name="base_width" value="0.4"/>
   <xacro:property name="base_height" value="0.02"/>
   <xacro:property name="top_length" value="0.246"/>
@@ -38,7 +38,10 @@
       </geometry>
     </collision>
+    <xacro:inertial_box mass="1.0" x="${base_length}" y="${base_width}" z="${base_height}">
+      <origin xyz="0.0 0.0 -${base_height/2}"/>
+    </xacro:inertial_box>
   </link>
   <!-- Top Plate -->
-  <joint name="top_joint" type="fixed">
+  <!-- <joint name="top_joint" type="fixed">
     <origin xyz="-${base_length/2 - top_length/2} ${base_width/2 - top_width/2} ${top_height}"/>
     <parent link="base_plate"/>
@@ -67,4 +70,4 @@
       </geometry>
     </collision>
-  </link>
+  </link> -->
 </robot>

File: description/bot.urdf.xacro (robot description, xacro)
@@ -1,6 +1,10 @@
 <?xml version="1.0"?>
-<robot xmlns:xacro="http://www.ros.org/wiki/xacro"  name="mangalyaan">
+<robot xmlns:xacro="http://www.ros.org/wiki/xacro"  name="Diff_Bot">
+    <!-- Base Plate -->
+    <xacro:include filename="inertial_macros.xacro"/>
     <!-- Base Plate -->
     <xacro:include filename="base.xacro"/>
+    <!-- Caster -->
+    <xacro:include filename="caster.xacro"/>
     <!-- Wheels -->
     <xacro:include filename="wheels.xacro"/>
@@ -8,4 +12,4 @@
     <xacro:include filename="lidar.xacro"/>
     <!-- ROS Control -->
-    <xacro:include filename="ros2_control.xacro"/>
+    <!-- <xacro:include filename="ros2_control.xacro"/> -->
 </robot>

File: description/lidar.xacro (robot description, xacro)
@@ -7,5 +7,5 @@
   <joint name="lidar_joint" type="fixed">
     <origin xyz="0 0 ${lidar_height/2}"/>
-    <parent link="top_plate"/>
+    <parent link="base_plate"/>
     <child link="lidar_link"/>
   </joint>
@@ -26,9 +26,7 @@
       </geometry>
     </collision>
-    <inertial>
-      <origin xyz="0 0 0"/>
-      <mass value="0.1"/>
-      <inertia ixx="0.0" ixy="0.0" ixz="0.0" iyy="0.0" iyz="0.0" izz="0.0"/>
-    </inertial>
+    <xacro:inertial_cylinder mass="0.1" radius="${lidar_radius}" length="${lidar_height}">
+      <origin xyz="0 0 ${lidar_height/2}"/>
+    </xacro:inertial_cylinder>
   </link>
   <gazebo reference="lidar_link">

File: description/wheels.xacro (robot description, xacro)
@@ -2,9 +2,7 @@
 <robot xmlns:xacro="http://www.ros.org/wiki/xacro">
   <!-- Variables -->
-  <xacro:property name="base_length" value="0.372" />
-  <xacro:property name="base_width" value="0.361" />
   <xacro:property name="wheel_radius" value="0.035" />
   <xacro:property name="wheel_width" value="0.04" />
-  <xacro:property name="wheel_gap" value="0.01" />
+  <xacro:property name="wheel_gap" value="0.009" />
   <!-- Wheel Macro -->
   <xacro:macro name="wheel" params="prefix parent x y z z_sign">
@@ -29,15 +27,13 @@
         </geometry>
       </collision>
-    <inertial>
-      <origin xyz="0 0 ${wheel_radius}"/>
-      <mass value="1"/>
-      <inertia ixx="0.0" ixy="0.0" ixz="0.0" iyy="0.0" iyz="0.0" izz="0.0"/>
-    </inertial>
+      <xacro:inertial_cylinder mass="0.1" radius="${wheel_radius}" length="${wheel_width}">
+        <origin xyz="0 0 0"/>
+      </xacro:inertial_cylinder>
     </link>
   </xacro:macro>
   <!-- Wheels -->
-  <xacro:wheel prefix="top_left" parent="base_plate" x="${base_width/2 - 0.03}" y="${base_length/2 + wheel_gap + wheel_width/2}" z="-0.04" z_sign="1"/>
-  <xacro:wheel prefix="top_right" parent="base_plate" x="${base_width/2 - 0.03}" y="-${base_length/2 + wheel_gap + wheel_width/2}" z="-0.04" z_sign="1"/>
-  <xacro:wheel prefix="bottom_left" parent="base_plate" x="-${base_width/2 - 0.03}" y="${base_length/2 + wheel_gap + wheel_width/2}" z="-0.04" z_sign="-1"/>
-  <xacro:wheel prefix="bottom_right" parent="base_plate" x="-${base_width/2 - 0.03}" y="-${base_length/2 + wheel_gap + wheel_width/2}" z="-0.04" z_sign="-1"/>
+  <!-- <xacro:wheel prefix="top_left" parent="base_plate" x="${base_width/2 - 0.03}" y="${base_length/2 + wheel_gap + wheel_width/2}" z="-0.04" z_sign="1"/>
+  <xacro:wheel prefix="top_right" parent="base_plate" x="${base_width/2 - 0.03}" y="-${base_length/2 + wheel_gap + wheel_width/2}" z="-0.04" z_sign="1"/> -->
+  <xacro:wheel prefix="bottom_left" parent="base_plate" x="-${base_length/2 - 0.013}" y="${base_width/2 + wheel_gap + wheel_width/2}" z="-0.04" z_sign="-1"/>
+  <xacro:wheel prefix="bottom_right" parent="base_plate" x="-${base_length/2 - 0.013}" y="-${base_width/2 + wheel_gap + wheel_width/2}" z="-0.04" z_sign="-1"/>
 </robot>
