Commit message: Rviz Visualization

File: description/caster.xacro (robot description, xacro)
@@ -9,5 +9,5 @@
             <parent link="${parent}"></parent>
             <child link="${prefix}_caster"></child>
-            <origin xyz="${x} ${y} ${z}" rpy="0 0 0" />
+            <origin xyz="${x} ${y} ${z}" rpy="${pi/2 * z_sign} 0 0" />
             <axis xyz="0 0 ${-1 * z_sign}" />
         </joint>
@@ -32,5 +32,5 @@
     </xacro:macro>
     <!-- Casters (two at the bottom) -->
-    <xacro:caster prefix="top_left" parent="base_plate" x="${base_length/2 - 0.01}" y="${base_width/2 - 0.01 }" z="${-caster_gap}" z_sign="1"/>
+    <xacro:caster prefix="top_left" parent="base_plate" x="${base_length/2 - 0.01}" y="${base_width/2 - 0.01 }" z="${-caster_gap}" z_sign="-1"/>
     <xacro:caster prefix="top_right" parent="base_plate" x="${base_length/2 - 0.01}" y="-${base_width/2 - 0.01 }" z="${-caster_gap}" z_sign="1"/>
 </robot>

File: description/wheels.xacro (robot description, xacro)
@@ -36,4 +36,4 @@
   <xacro:wheel prefix="top_right" parent="base_plate" x="${base_width/2 - 0.03}" y="-${base_length/2 + wheel_gap + wheel_width/2}" z="-0.04" z_sign="1"/> -->
   <xacro:wheel prefix="bottom_left" parent="base_plate" x="-${base_length/2 - 0.013}" y="${base_width/2 + wheel_gap + wheel_width/2}" z="-0.04" z_sign="-1"/>
-  <xacro:wheel prefix="bottom_right" parent="base_plate" x="-${base_length/2 - 0.013}" y="-${base_width/2 + wheel_gap + wheel_width/2}" z="-0.04" z_sign="-1"/>
+  <xacro:wheel prefix="bottom_right" parent="base_plate" x="-${base_length/2 - 0.013}" y="-${base_width/2 + wheel_gap + wheel_width/2}" z="-0.04" z_sign="1"/>
 </robot>
